Commit message: feat: switch to YOLOv8 for human detection, replace Haar cascade

File: src/warehouse_amr/urdf/warehouse_amr.urdf.xacro (robot description, xacro)
@@ -101,5 +101,5 @@
     <parent link="base_link"/>
     <child  link="depth_camera_link"/>
-    <origin xyz="${base_length/2} 0 ${base_height/2 + 0.05}" rpy="0 0 0"/>
+    <origin xyz="${base_length/2} 0 ${base_height/2 + 0.05}" rpy="0 -0.2094 0"/>
   </joint>
   <link name="depth_camera_optical_frame"/>
